Commit message: Add files via upload

File: mod5/ex03/circle_movement/description/gazebo.urdf.xacro (robot description, xacro)
@@ -24,9 +24,9 @@
             filename="gz-sim-diff-drive-system"
             name="gz::sim::systems::DiffDrive">
-            <left_joint>wheel_2_joint</left_joint>
-            <right_joint>wheel_1_joint</right_joint>
+            <left_joint>wheel_1_joint</left_joint>
+            <right_joint>wheel_2_joint</right_joint>
             <child_frame_id>kak/base_link</child_frame_id>
-            <wheel_separation>2.0</wheel_separation>
-            <wheel_radius>0.35</wheel_radius>
+            <wheel_separation>0.35</wheel_separation>
+            <wheel_radius>0.1</wheel_radius>
             <odom_publish_frequency>10</odom_publish_frequency>
         </plugin>

File: mod5/ex03/circle_movement/description/kak.urdf.xacro (robot description, xacro)
@@ -65,5 +65,5 @@
       </geometry>
     </collision>
-    <xacro:cylinder_inertia m="0.7" r="1.0" h="0.07"/>
+    <xacro:cylinder_inertia m="0.5" r="1.0" h="0.07"/>
   </link>
   <joint name="stol_joint" type="fixed">
@@ -85,5 +85,5 @@
       </geometry>
     </collision>
-    <xacro:box_inertia m="0.5" w="0.52" d="0.56" h="0.685"/>
+    <xacro:box_inertia m="5" w="0.52" d="0.56" h="0.685"/>
   </link>
   <joint name="vaza_joint" type="fixed">
@@ -104,5 +104,5 @@
       </geometry>
     </collision>
-    <xacro:box_inertia m="0.5" w="0.42" d="0.46" h="0.585"/>
+    <xacro:box_inertia m="5" w="0.42" d="0.46" h="0.585"/>
   </link>
   <joint name="zemlya_joint" type="fixed">
@@ -195,5 +195,6 @@
   <xacro:igli prefix="5" z_high = "0.7225" a_long = "0.05" b_weight = "0.45" />
   <xacro:igli prefix="6" z_high = "0.7225" a_long = "0.45" b_weight = "0.05" />
-    <link name="wheel_1">
+  <xacro:macro name = "wheel" params = "prefix x">
+    <link name="wheel_${prefix}">
       <visual>
        <origin xyz="0 0 0" rpy="1.56 0 0"/>
@@ -211,33 +212,14 @@
       <xacro:cylinder_inertia m="0.7" r="0.35" h="0.15"/>
     </link>
-    <joint name="wheel_1_joint" type="continuous">
-      <parent link="base_link"/>
-      <child link="wheel_1"/>
-      <origin xyz="-0.5 0.9 -0.45" rpy="0 -1.56 0"/>
+    <joint name="wheel_${prefix}_joint" type="continuous">
+      <parent link="stol"/>
+      <child link="wheel_${prefix}"/>
+      <origin xyz="${x} -0.5 -0.45" rpy="0 0 1.56"/>
       <axis xyz="0 1 0"/>
     </joint>
-    <link name="wheel_2">
-      <visual>
-       <origin xyz="0 0 0" rpy="1.56 0 0"/>
-        <geometry>
-          <cylinder radius="0.35" length="0.15"/>
-	</geometry>
-        <material name="Blue"/>
-      </visual>
-      <collision>
-        <origin xyz="0 0 0" rpy="${pi/2} 0 0"/>
-        <geometry>
-          <cylinder radius="0.35" length="0.15"/>
-        </geometry>
-      </collision>
-      <xacro:cylinder_inertia m="0.7" r="0.35" h="0.15"/>
-    </link>
-    <joint name="wheel_2_joint" type="continuous">
-      <parent link="base_link"/>
-      <child link="wheel_2"/>
-      <origin xyz="-0.5 -0.9 -0.45" rpy="0 1.56 0"/>
-      <axis xyz="0 1 0"/>
-    </joint>
-  <link name="wheel_center">
+  </xacro:macro>
+  <xacro:wheel prefix="1" x = "0.9"/>
+  <xacro:wheel prefix="2" x = "-0.9"/>
+  <link name="weel_center">
     <visual>
       <geometry>
@@ -251,13 +233,13 @@
       </geometry>
     </collision>
-    <xacro:sphere_inertia m="1.0" r="0.2"/>
-  </link>
-  <joint name="wheel_center_joint" type="fixed">
-    <parent link="base_link"/>
-    <child link="wheel_center"/>
-    <origin xyz="0.8 0 -0.6" rpy="0 1.56 0"/>
-    <!--axis xyz="0 1 0"/-->
-  </joint>
-   <gazebo reference="wheel_center">
+    <xacro:sphere_inertia m="0.3" r="0.2"/>
+  </link>
+  <joint name="weel_center_joint" type="continuous">
+    <parent link="stol"/>
+    <child link="weel_center"/>
+    <origin xyz="0 0.6 -0.6" rpy="0 0 0"/>
+  </joint>
+   <gazebo reference="weel_center">
+      <material>Orange</material>
       <mu1 value="0.001"/>
       <mu2 value="0.001"/>
